File: eagle/laser-driver/laser-driver.brd (EAGLE design)
At the start: 68.6 x 37.2 mm, 49 parts, among them IC1 74HC589D, IC2 74HC589D, IC3 TC7660SOIC8, T1 2N7002E, T2 2N7002E, U1 AD8041ARZ, U2 SN74HC163NSR, U3 SN74LVC1G14DBVT, U4 MCP6291T-E/OT, U5 SN74AHCT1G08DCKR, U6 SN74LVC1G17DBVR

Commit message: Update PCBs, schematics, processed jobs, etc.
Parts:
- removed D1: VTB8441BH, mulabs:VTB8441BH
- removed N(SYNC): TPB1,27, testpad:B1,27
- removed U1: AD8041ARZ, Analog Devices_By_element14_Batch_1:SOIC127P600X175-8N
- removed U3: SN74LVC1G14DBVT, Texas Instruments_By_element14_Batch_1:SOT95P280X145-5N
- removed U4: MCP6291T-E/OT, Microchip_By_element14_Batch_1:SOT95P320X145-5N
- removed U5: SN74AHCT1G08DCKR, Texas Instruments_By_element14_Batch_1:SOT65P210X110-5N
- removed U6: SN74LVC1G17DBVR, Texas Instruments_By_element14_Batch_1:SOT95P280X145-5N
- added !RESET, COMP: TPB1,27, testpad:B1,27
- added C14, C15, C16, C18, C20, C24: 10nF, rcl:C1206
- added C17, C19, C23: 1µ, rcl:C1206
- added C21: 100nF, rcl:C1206
- added C22: 10µ, rcl:A/3216-18R
- added C25: 100µF, rcl:D/7343-31R
- added C26, C29, C30: 100nF, rcl:C0603
- added C27, C28: 220µ, rcl:153CLV-0605
- added C31: 100n, rcl:C0603
- added C32: 22pF, rcl:C0603
- added D2: 15MQ040NTR, SparkFun:SMA-DIODE
- added D3: VTB8441BH, mulabs:VTB8441BH
- added IC4: AD8041R, analog-devices:SO8
- added IC5: 74LVC1G17DBV, 74xx-little-de:SOT23-5
- added IC6: 74LVC1G14DBV, 74xx-little-de:SOT23-5
- added IC7: 74AHCT1G08DCK, 74xx-little-de:SC70-5
- added LED1, LED2: (no value), led:CHIPLED_0805
- added R16: 820Ω, rcl:R0603
- added R17: 10kΩ, rcl:R0603
- added R18: 270Ω, rcl:R0603
- added R19: 10k, rcl:R0603
- added R20: 100k, pot:SM-42/43B
- added R21: 100kΩ+, rcl:R0603
- added R22, R23: 300Ω, rcl:R0603
- added R24: 1kΩ, pot:3223G
- added SJ1: CURRENT MEASURE, SparkFun:SJ_2S-NO
- added T3: 2N7002E, nxp_60:SOT23
- added TVS2: 6V, supressor:TVS0805
- added U7: MCP6561T, mulabs:SOT23-5
- added U8: MCP6291T-E/OT, mulabs:SOT23-5
- C13: device rcl:C1206 -> rcl:C0603
- C5: value 100pF -> 10nF; device rcl:C1206 -> rcl:C0603
- C6, C7: value 50pF -> 10nF
- R1, R12, R4, R9: device rcl:R1206 -> rcl:R0603
- R13: value 1k -> 10k; device rcl:R1206 -> rcl:R0603
- R14: value 100k -> 150Ω; device rcl:R1206 -> rcl:R0603
- R2: value 120Ω -> 1kΩ; device rcl:R1206 -> rcl:R0603
- R3: value 5k -> 1kΩ; device pot:3223W -> pot:SM-42/43B
- R5: value 1k -> 5.1kΩ; device rcl:R1206 -> rcl:R0603
- R6: value 10Ω -> 12Ω; device rcl:R1206 -> rcl:R0603
- R7: value 3.3kΩ -> 100 Ω; device rcl:R1206 -> rcl:R0603
- R8: value 6.8kΩ -> 100 Ω; device rcl:R1206 -> rcl:R0603
- moved C8 38.2 mm to (17.7, 37.2), flipped to the bottom, turned to 0 degrees
- moved R1 34.1 mm to (27.8, 33.5), turned to 180 degrees
- moved C3 29.2 mm to (61.1, 14.1), flipped to the bottom, turned to 270 degrees
- moved C7 28.4 mm to (56.9, 33.4)
- moved PD 20.0 mm to (27.9, 24.8), turned to 90 degrees
- moved C2 19.2 mm to (56.9, 35.9), turned to 0 degrees
- moved R13 18.3 mm to (12.2, 27.8)
- moved CLK 12.7 mm to (30.0, 7.62)
- moved R2 12.4 mm to (43.3, 36.3), turned to 270 degrees
- moved T2 11.5 mm to (33.0, 32.9), turned to 0 degrees
- moved C6 11.0 mm to (17.7, 34.5), flipped to the bottom
- moved C9 11.0 mm to (9.40, 11.6)
- moved R6 10.2 mm to (49.9, 38.1), turned to 180 degrees
- moved LD-EN 8.89 mm to (59.8, 38.0)
- moved R8 8.54 mm to (67.4, 13.3), turned to 90 degrees
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Connections:
- new net N$13: C15.1, R1.1, R8.2, T2.1
- new net N$28: R16.1, T2.2
- new net N$29: R18.1, T3.2
- new net N$30: R13.2, R19.1, U8.3
- new net N$31: D2.C, SJ1.1, TVS2.2, U$1.1
- new net N$32: C5.1, PD.TP, R12.2, U7.4
- new net N$33: LED1.C, R22.2
- new net N$34: LED2.C, R23.2
- new net N$35: IC4.2, R2.2
- new net N$36: R14.2, R24.1
- net GND: now also C14.2, C15.2, C16.2, C17.2, C18.2, C19.2, C20.2, C22.+, C23.1, C24.1, C25.-, C26.2, C27.-, C28.-, C29.2, C30.2, C31.2, C32.2, C6.2, C7.2, IC5.3, IC6.3, IC7.3, R13.1, R16.2, R17.2, R18.2, R20.3, R22.1, R23.1, R3.3, U7.2, U8.2; no longer D1.A, R2.1, R3.1, T2.2, U3.3, U4.3, U5.3, U6.3
- net N$1: now also IC4.8; no longer U1.8
- net N$11: now also !RESET.TP; no longer N(SYNC).TP
- net N$12: now also R21.1, U7.1; no longer C5.1, PD.TP, R12.2
- net N$15: now also C21.2
- net N$16: now also IC7.4; no longer U5.4
- net N$17: now also IC6.4, IC7.2; no longer U3.4, U5.2
- net N$19: now also COMP.TP, R20.2, R21.2, U7.3; no longer C6.2, C7.2, R13.2, U4.4
- net N$2: now also C32.1, R3.1, T3.3; no longer R2.2, R3.3
- net N$20: now also IC6.2; no longer U3.2
- net N$21: now also D3.A, U8.4; no longer D1.K, R13.1
- net N$23: now also R24.2, R24.3, U8.1; no longer C6.1, C7.1, R14.2, U4.1
- net N$24: now also IC5.2; no longer U6.2
- net N$25: now also C21.1
- net N$27: now also IC5.4, IC7.1; no longer U5.1, U6.4
- net N$3: now also IC4.6; no longer U1.6
- net N$5: now also D2.A, TVS2.1
- net N$6: now also R2.1; no longer U1.2
- net N$8: now also IC4.3; no longer U1.3
- net N$9: now also C14.1, R17.1, T3.1; no longer R1.1, R8.2, T2.1
- net VCC: now also C16.1, C17.1, C18.1, C19.1, C20.1, C25.+, C26.1, C27.+, C28.+, C29.1, C30.1, C31.1, C6.1, C7.1, D3.K, IC4.7, IC5.5, IC6.5, IC7.5, LED1.A, LED2.A, R19.2, R20.1, SJ1.2, U7.5, U8.5; no longer U$1.1, U1.7, U3.5, U4.5, U5.5, U6.5
- net VSS: now also C22.-, C23.2, C24.2, IC4.4; no longer U1.4, U4.2
Routing:
- net VCC: track 154.1 -> 266.1 mm, vias 3 -> 10
- net N$13: track 0.00 -> 59.1 mm, vias 0 -> 2
- net N$31: track 0.00 -> 12.6 mm
- net N$10: track 16.2 -> 4.29 mm
- net N$24: track 14.2 -> 5.16 mm
- net N$32: track 0.00 -> 8.83 mm
- net N$21: track 14.2 -> 5.56 mm
- net N$27: track 9.36 -> 1.90 mm
- net N$9: track 66.3 -> 59.3 mm
- net N$2: track 49.3 -> 42.4 mm
- net N$30: track 0.00 -> 6.79 mm
- net N$4: track 15.5 -> 8.81 mm
- net VSS: track 69.4 -> 76.1 mm
- net GND: track 0.00 -> 6.07 mm, vias 7 -> 8
- net N$36: track 0.00 -> 5.83 mm
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Other:
- board size 68.6 x 37.2 mm -> 68.6 x 37.8 mm
- board text added: "1"
- board text added: "LASER DRIVER v3"
- board text added: "V3"
- board text added: "mulabs.org"

Commit message: PLL acquires lock
Parts:
- added R25, R26: 10kΩ, rcl:R0603
- R20: value 100k -> 5kΩ
Connections:
- new net N$37: C31.1, R20.1, R25.2
- new net N$38: R20.2, R26.2
- net N$19: now also R26.1; no longer R20.2
- net VCC: now also R25.1; no longer C31.1, R20.1
Routing:
- net N$19: track 14.5 -> 8.18 mm
- net VCC: track 266.1 -> 260.0 mm
Changed lines of the file:
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@@
 <?xml version="1.0" encoding="utf-8"?>
 <!DOCTYPE eagle SYSTEM "eagle.dtd">
-<eagle version="7.5.0">
+<eagle version="7.7.0">
 <drawing>
 <settings>
@@
 <grid distance="0.01" unitdist="mm" unit="mm" style="lines" multiple="1" display="no" altdistance="0.005" altunitdist="inch" altunit="inch"/>
 <layers>
-<layer number="1" name="Top" color="4" fill="1" visible="no" active="yes"/>
+<layer number="1" name="Top" color="4" fill="1" visible="yes" active="yes"/>
 <layer number="2" name="Route2" color="1" fill="3" visible="no" active="no"/>
 <layer number="3" name="Route3" color="4" fill="3" visible="no" active="no"/>
 <layer number="14" name="Route14" color="1" fill="6" visible="no" active="no"/>
 <layer number="15" name="Route15" color="4" fill="6" visible="no" active="no"/>
-<layer number="16" name="Bottom" color="1" fill="1" visible="no" active="yes"/>
+<layer number="16" name="Bottom" color="1" fill="1" visible="yes" active="yes"/>
 <layer number="17" name="Pads" color="2" fill="1" visible="yes" active="yes"/>
 <layer number="18" name="Vias" color="2" fill="1" visible="yes" active="yes"/>
-<layer number="19" name="Unrouted" color="6" fill="1" visible="no" active="yes"/>
+<layer number="19" name="Unrouted" color="6" fill="1" visible="yes" active="yes"/>
 <layer number="20" name="Dimension" color="15" fill="1" visible="yes" active="yes"/>
 <layer number="21" name="tPlace" color="7" fill="1" visible="yes" active="yes"/>
-<layer number="22" name="bPlace" color="7" fill="1" visible="no" active="yes"/>
+<layer number="22" name="bPlace" color="7" fill="1" visible="yes" active="yes"/>
 <layer number="23" name="tOrigins" color="15" fill="1" visible="yes" active="yes"/>
-<layer number="24" name="bOrigins" color="15" fill="1" visible="no" active="yes"/>
-<layer number="25" name="tNames" color="7" fill="1" visible="no" active="yes"/>
-<layer number="26" name="bNames" color="7" fill="1" visible="no" active="yes"/>
-<layer number="27" name="tValues" color="7" fill="1" visible="yes" active="yes"/>
+<layer number="24" name="bOrigins" color="15" fill="1" visible="yes" active="yes"/>
+<layer number="25" name="tNames" color="7" fill="1" visible="yes" active="yes"/>
+<layer number="26" name="bNames" color="7" fill="1" visible="yes" active="yes"/>
+<layer number="27" name="tValues" color="7" fill="1" visible="no" active="yes"/>
 <layer number="28" name="bValues" color="7" fill="1" visible="no" active="yes"/>
 <layer number="29" name="tStop" color="7" fill="3" visible="no" active="yes"/>
@@
 <layer number="37" name="tTest" color="7" fill="1" visible="no" active="yes"/>
 <layer number="38" name="bTest" color="7" fill="1" visible="no" active="yes"/>
-<layer number="39" name="tKeepout" color="4" fill="11" visible="no" active="yes"/>
-<layer number="40" name="bKeepout" color="1" fill="11" visible="no" active="yes"/>
-<layer number="41" name="tRestrict" color="4" fill="10" visible="no" active="yes"/>
-<layer number="42" name="bRestrict" color="1" fill="10" visible="no" active="yes"/>
-<layer number="43" name="vRestrict" color="2" fill="10" visible="no" active="yes"/>
+<layer number="39" name="tKeepout" color="4" fill="11" visible="yes" active="yes"/>
+<layer number="40" name="bKeepout" color="1" fill="11" visible="yes" active="yes"/>
+<layer number="41" name="tRestrict" color="4" fill="10" visible="yes" active="yes"/>
+<layer number="42" name="bRestrict" color="1" fill="10" visible="yes" active="yes"/>
+<layer number="43" name="vRestrict" color="2" fill="10" visible="yes" active="yes"/>
 <layer number="44" name="Drills" color="7" fill="1" visible="no" active="yes"/>
 <layer number="45" name="Holes" color="7" fill="1" visible="no" active="yes"/>
@@
 <layer number="50" name="dxf" color="7" fill="1" visible="no" active="no"/>
 <layer number="51" name="tDocu" color="7" fill="1" visible="yes" active="yes"/>
-<layer number="52" name="bDocu" color="7" fill="1" visible="no" active="yes"/>
+<layer number="52" name="bDocu" color="7" fill="1" visible="yes" active="yes"/>
 <layer number="53" name="tGND_GNDA" color="7" fill="9" visible="no" active="no"/>
 <layer number="54" name="bGND_GNDA" color="1" fill="9" visible="no" active="no"/>
@@
 <attribute name="VALUE" x="17.385" y="24.918" size="0.6096" layer="27" rot="R180"/>
 </element>
-<element name="R20" library="pot" package="SM-42/43B" value="100k" x="38.354" y="23.114" smashed="yes" rot="R180">
+<element name="R20" library="pot" package="SM-42/43B" value="5kΩ" x="38.354" y="23.114" smashed="yes" rot="R180">
 <attribute name="NAME" x="37.298" y="24.038" size="0.6096" layer="25" rot="R270"/>
 <attribute name="VALUE" x="39.532" y="22.75" size="0.6096" layer="27" rot="R180"/>
@@
 <attribute name="VALUE" x="44.323" y="22.479" size="0.0254" layer="27"/>
 </element>
+<element name="R25" library="rcl" package="R0603" value="10kΩ" x="1.63" y="0.08"/>
+<element name="R26" library="rcl" package="R0603" value="10kΩ" x="1.63" y="-4.67"/>
 </elements>
 <signals>
@@
 <wire x1="19.05" y1="34.541" x2="19.053" y2="34.544" width="0.254" layer="16"/>
 <wire x1="41.636871875" y1="16.764" x2="41.656" y2="16.744871875" width="0.254" layer="16"/>
-<contactref element="C31" pad="1"/>
 <wire x1="20.1676" y1="29.3878" x2="22.2758" y2="29.3878" width="0.4064" layer="1"/>
 <contactref element="C30" pad="1"/>
@@
 <wire x1="30.734" y1="29.845" x2="32.512" y2="29.845" width="0.4064" layer="1"/>
 <wire x1="32.512" y1="29.845" x2="34.163" y2="28.194" width="0.4064" layer="1"/>
-<contactref element="R20" pad="1"/>
-<wire x1="35.754" y1="21.964" x2="39.377" y2="21.964" width="0.254" layer="1"/>
 <wire x1="39.377" y1="21.964" x2="39.751" y2="21.59" width="0.254" layer="1"/>
 <wire x1="39.751" y1="21.59" x2="41.275" y2="21.59" width="0.254" layer="1"/>
@@
 <wire x1="26.797" y1="21.5392" x2="26.67" y2="21.6662" width="0.4064" layer="1"/>
 <wire x1="26.797" y1="21.5392" x2="26.797" y2="20.281" width="0.4064" layer="1"/>
-<wire x1="26.797" y1="20.281" x2="25.019" y2="18.503" width="0.4064" layer="1"/>
 <wire x1="18.796" y1="21.336" x2="18.161" y2="21.971" width="0.4064" layer="1"/>
 <wire x1="18.161" y1="21.971" x2="18.161" y2="23.622" width="0.4064" layer="1"/>
@@
 <wire x1="16.383" y1="23.622" x2="16.383" y2="27.429" width="0.4064" layer="16"/>
 <wire x1="18.161" y1="23.622" x2="16.383" y2="23.622" width="0.4064" layer="16"/>
+<contactref element="R25" pad="1"/>
+<wire x1="0.78" y1="0.08" x2="8.382" y2="9.873" width="0" layer="19" extent="1-16"/>
 </signal>
 <signal name="N$2">
@@
 </signal>
 <signal name="N$19">
-<contactref element="R20" pad="2"/>
 <contactref element="R21" pad="2"/>
 <contactref element="U7" pad="3"/>
 <contactref element="COMP" pad="TP"/>
 <wire x1="41.081" y1="23.241" x2="44.958" y2="23.241" width="0.254" layer="1"/>
-<wire x1="41.081" y1="23.241" x2="40.954" y2="23.114" width="0.254" layer="1"/>
 <wire x1="30.7086" y1="23.5458" x2="33.3638" y2="23.5458" width="0.254" layer="1"/>
 <wire x1="33.3638" y1="23.5458" x2="33.401" y2="23.583" width="0.254" layer="1"/>
-<wire x1="40.954" y1="23.114" x2="34.798" y2="23.114" width="0.254" layer="1"/>
 <wire x1="34.798" y1="23.114" x2="34.329" y2="23.583" width="0.254" layer="1"/>
 <wire x1="33.401" y1="23.583" x2="34.329" y2="23.583" width="0.254" layer="1"/>
+<contactref element="R26" pad="1"/>
+<wire x1="34.798" y1="23.114" x2="41.081" y2="23.241" width="0" layer="19" extent="1-1"/>
+<wire x1="0.78" y1="-4.67" x2="30.7086" y2="23.5458" width="0" layer="19" extent="1-1"/>
 </signal>
 <signal name="N$33">
@@
 <wire x1="21.885" y1="33.652" x2="21.885" y2="32.725" width="0.254" layer="1"/>
 </signal>
+<signal name="N$37">
+<contactref element="C31" pad="1"/>
+<contactref element="R20" pad="1"/>
+<contactref element="R25" pad="2"/>
+<wire x1="25.019" y1="18.503" x2="35.754" y2="21.964" width="0" layer="19" extent="1-1"/>
+<wire x1="2.48" y1="0.08" x2="25.019" y2="18.503" width="0" layer="19" extent="1-1"/>
+</signal>
+<signal name="N$38">
+<contactref element="R20" pad="2"/>
+<contactref element="R26" pad="2"/>
+<wire x1="2.48" y1="-4.67" x2="40.954" y2="23.114" width="0" layer="19" extent="1-1"/>
+</signal>
 </signals>
