File: eagle/MCU/mcu.sch (EAGLE design)
At the start: 87 parts, among them IC1 HCT4046A, IC10 LD117ADT50TR, IC2 AZ1117-3.3, IC3 4059D, IC4 AZ1086, IC5 74AHCT1G08DCK, IC7 74LVX4245TSSOP24W, IC8 74LVX4245TSSOP24W, IC9 74LVX4245TSSOP24W, T1 2N7002E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

Commit message: PLL acquires lock
Parts:
- removed R27, R30: 10kΩ, rcl:R-EU_R0603
- added R18: 5kΩ, rcl:R-EU_R0603
- added R19: 10kΩ, rcl:R-EU_R0603
- added T6: BC857, transistor:BC857C-PNP-SOT23-BEC
- R8: value 500Ω -> 100Ω
- R9: value 1kΩ -> 10kΩ
- T1: value 2N7002E -> BC817; device nxp_60:2N7002E -> transistor:BC817-40-NPN-SOT23-BEC
- renumbered CTR_OUT to DIVIDER_OUT
Connections:
- removed net DIVIDER_OUT1: IC5A.O, PLL_IN.TP, R27.1, T1.S
- new net DIVIDER_OUT_IF_NOT_USING_EVOUT_PD4: U1.(OC1B/XCK1/MOSI)PF5
- new net N$41: R8.2, T1.B
- new net N$42: R19.1, T1.C
- new net PLL_IN_3V3: IC5A.O, PLL_IN.TP, R8.1
- new net PLL_IN_5V: IC1A.CIN, R9.2, T6.C
- net DIVIDER_OUT: now also U1.(OC1A/!SS!)PD4; no longer IC3.OUT, U1.(OC1B/XCK1/MOSI)PF5
- net GND: now also T1.E; no longer IC9.B4
- net LM_CLK: now also U1.(OC0A/SDA)PD0
- net LM_SYNC: no longer R8.2
- net N$2: now also R18.1, R19.2, T6.B; no longer IC1A.CIN, R30.1, T1.D
- net N$77: no longer R8.1, R9.2
- net VCC/3.3V: no longer C12P.2, IC3.VDD, R27.2, T1.G
- net VCC/5V: now also C12P.2, IC3.VDD, R18.2, T6.E; no longer R30.2
Other:
- note added: "TODO - LM_SYNC go through level-converter"
- note added: "TODO laser-enable should not collide with UART TXD"
- note added: "TODO usun licznik"
- moved on the sheet: R8, R9

Commit message: Next version
Connections:
- removed net DIVIDER_OUT_IF_NOT_USING_EVOUT_PD4: U1.(OC1B/XCK1/MOSI)PF5
- new net PD4: U1.(OC1A/!SS!)PD4
- net DIVIDER_OUT: now also U1.(OC1B/XCK1/MOSI)PF5; no longer U1.(OC1A/!SS!)PD4
Other:
- moved on the sheet: R18, R19, R8, R9, T1, T6
